File: Hardware/enciso y mateo lopez/oficialenciso y mateo lopez.kicad_pcb (KiCad board)
At the start: 2 copper layers, 14 parts, among them K1 SANYOU_SRD_Form_C, K2 SANYOU_SRD_Form_C, K3 SANYOU_SRD_Form_C, K4 SANYOU_SRD_Form_C, Q1 BC547, U1 ESP32-WROOM-32

Commit message: ESQUEMA GOD
Parts:
- removed C1: 10µF, Capacitor_THT:CP_Radial_D10.0mm_P5.00mm
- removed C2: 100nF, Capacitor_THT:CP_Radial_D10.0mm_P5.00mm
- added D2: D, Diode_THT:D_5W_P12.70mm_Horizontal, F.Cu at (205.8, 70.5)
- added D3: D, Diode_THT:D_5W_P12.70mm_Horizontal, F.Cu at (208.7, 87.0)
- added D4: D, Diode_THT:D_5W_P12.70mm_Horizontal, F.Cu at (206.8, 114.0)
- added Q2: BC547, Package_TO_SOT_THT:TO-92_Inline, F.Cu at (171.0, 70.0)
- added Q3: BC547, Package_TO_SOT_THT:TO-92_Inline, F.Cu at (176.0, 89.0)
- added Q4: BC547, Package_TO_SOT_THT:TO-92_Inline, F.Cu at (179.0, 110.5)
- added R10: 220, Resistor_SMD:R_0805_2012Metric, F.Cu at (193.1, 109.5)
- added R11: 1k, Resistor_SMD:R_0805_2012Metric, F.Cu at (198.2, 110.0)
- added R12: 10k, Resistor_SMD:R_0805_2012Metric, F.Cu at (194.4, 115.0)
- added R6: 10k, Resistor_SMD:R_0805_2012Metric, F.Cu at (195.3, 71.0)
- added R7: 220, Resistor_SMD:R_0805_2012Metric, F.Cu at (186.6, 87.5)
- added R8: 1k, Resistor_SMD:R_0805_2012Metric, F.Cu at (194.4, 89.0)
- added R9: 10k, Resistor_SMD:R_0805_2012Metric, F.Cu at (197.4, 86.5)
- added U2: ESP32-WROOM-32, RF_Module:ESP32-WROOM-32, F.Cu at (103.7, 81.6)
- added U2.1: PC817, Package_DIP:DIP-4_W7.62mm, F.Cu at (154.2, 72.2)
- added U3: PC817, Package_DIP:DIP-4_W7.62mm, F.Cu at (152.7, 87.7)
- added U4: PC817, Package_DIP:DIP-4_W7.62mm, F.Cu at (155.2, 108.7)
- R1, R4: value 1k -> 220
- R2: value 10k -> 1k
- R3: value 1k -> 10k
- U1: value ESP32-WROOM-32 -> PC817; footprint RF_Module:ESP32-WROOM-32 -> Package_DIP:DIP-4_W7.62mm
- moved K1 163.6 mm to (233.3, 42.5)
- moved R1 112.6 mm to (188.6, 43.0), turned to 0 degrees
- moved D1 111.5 mm to (204.2, 43.0)
- moved R2 109.9 mm to (186.5, 49.5), turned to 0 degrees
- moved R3 89.5 mm to (194.6, 45.5)
- moved R5 87.6 mm to (191.7, 67.0)
- moved K2 87.5 mm to (233.3, 64.5)
- moved R4 86.3 mm to (189.1, 70.5)
- moved K3 85.6 mm to (232.8, 87.0)
- moved K4 83.9 mm to (232.5, 111.5)
- moved Q1 78.8 mm to (172.0, 43.5)
- moved U1 74.0 mm to (155.7, 43.7)
Connections:
- D1 pad 1: NO -> +5V
- D1 pad 2: COM -> Net-(D1-A)
- K1 pad 1: 5V -> COM
- K1 pad 2: GND -> Net-(D1-A)
- K1 pad 3: IN -> NO
- K1 pad 4: COM -> NC
- K1 pad 5: NO -> +5V
- K2 pad 1: 5V -> COM
- K2 pad 2: GND -> Net-(D2-A)
- K2 pad 3: unconnected-(K2-Pad3) -> NO
- K2 pad 4: unconnected-(K2-Pad4) -> NC
- K2 pad 5: unconnected-(K2-Pad5) -> +5V
- K3 pad 1: 5V -> COM
- K3 pad 2: GND -> Net-(D3-A)
- K3 pad 3: unconnected-(K3-Pad3) -> NO
- K3 pad 4: unconnected-(K3-Pad4) -> NC
- K3 pad 5: unconnected-(K3-Pad5) -> +5V
- K4 pad 1: 5V -> COM
- K4 pad 2: GND -> Net-(D4-A)
- K4 pad 3: unconnected-(K4-Pad3) -> NO
- K4 pad 4: unconnected-(K4-Pad4) -> NC
- K4 pad 5: unconnected-(K4-Pad5) -> +5V
- Q1 pad 1: IN -> Net-(D1-A)
- Q1 pad 2: BASE -> Net-(Q1-B)
- R1 pad 1: GPIO -> INPUT
- R1 pad 2: BASE -> Net-(R1-Pad2)
- R2 pad 1: GPIO2 -> Net-(R2-Pad1)
- R2 pad 2: GND -> Net-(Q1-B)
- R3 pad 1: unconnected-(R3-Pad1) -> Net-(Q1-B)
- R4 pad 1: unconnected-(R4-Pad1) -> INPUT2
- R4 pad 2: GND -> Net-(R4-Pad2)
- R5 pad 1: unconnected-(R5-Pad1) -> Net-(R5-Pad1)
- R5 pad 2: GND -> Net-(Q2-B)
- U1 pad 1: GND -> Net-(R1-Pad2)
- U1 pad 2: VCC -> GND
- U1 pad 3: unconnected-(U1-EN-Pad3) -> Net-(R2-Pad1)
- U1 pad 4: unconnected-(U1-SENSOR_VP-Pad4) -> +5V
Routing:
- net 5V: track 80.5 -> 0.00 mm
- net GND: track 77.2 -> 0.00 mm
- net IN: track 27.2 -> 0.00 mm
- net GPIO: track 1.17 -> 0.00 mm
